Commit message: Changed some parameters of the URDF

File: comau_ros2_client/comau_description/racer5-cobot_description/urdf/racer5-cobot/racer5-cobot.urdf.xacro (robot description, xacro)
@@ -17,4 +17,5 @@
       </inertial>
       <visual>
+        <origin xyz="0 0 0" rpy="0 0 0" />
         <geometry>
           <mesh filename="package://racer5-cobot_description/meshes/racer5-cobot/base_link.STL" />
@@ -36,5 +37,5 @@
       </inertial>
       <visual>
-        <origin xyz="0 0 0" rpy="0 0 0" />
+        <origin xyz="0 0 -0.050" rpy="0 0 0" />
         <geometry>
           <mesh filename="package://racer5-cobot_description/meshes/racer5-cobot/Link1.STL" />
@@ -50,8 +51,8 @@
     </link>
     <joint name="${prefix}joint_1" type="revolute">
-      <origin xyz="0 0 0.1895" rpy="0 0 0" />
+      <origin xyz="0 0 0.242" rpy="0 0 0" />
       <parent link="base_link" />
       <child link="link_1" />
-      <axis xyz="0 0 1" />
+      <axis xyz="0 0 -1" />
       <limit lower="-2.966" upper="2.966" effort="100000.00" velocity="20.00" />
     </joint>
@@ -77,9 +78,9 @@
     </link>
     <joint name="${prefix}joint_2" type="revolute">
-      <origin xyz="0.05 0 0.1755" rpy="0 0 0" />
+      <origin xyz="0.05 0 0.123" rpy="0 0 0" />
       <parent link="link_1" />
       <child link="link_2" />
-      <axis xyz="0 -1 0" />
-      <limit lower="-1.99" upper="1.116" effort="100000.00" velocity="20.00" />
+      <axis xyz="0 1 0" />
+      <limit lower="-1.116" upper="1.99" effort="100000.00" velocity="20.00" />
     </joint>
     <link name="${prefix}link_3">
@@ -90,5 +91,5 @@
       </inertial>
       <visual>
-        <origin xyz="0 0 0" rpy="0 0 0" />
+        <origin xyz="0 0 0" rpy="0 0 3.14" />
         <geometry>
           <mesh filename="package://racer5-cobot_description/meshes/racer5-cobot/Link3.STL" />
@@ -104,8 +105,8 @@
     </link>
     <joint name="${prefix}joint_3" type="revolute">
-      <origin xyz="0 0 0.37" rpy="0 0 0" />
+      <origin xyz="0 0 0.37" rpy="0 0 3.14" />
       <parent link="link_2" />
       <child link="link_3" />
-      <axis xyz="0 -1 0" />
+      <axis xyz="0 1 0" />
       <limit lower="-2.62" upper="1.483" effort="100000.00" velocity="20.00" />
     </joint>
@@ -117,5 +118,5 @@
       </inertial>
       <visual>
-        <origin xyz="0 0 0" rpy="0 0 0" />
+        <origin xyz="0 0 0" rpy="0 0 3.14" />
         <geometry>
           <mesh filename="package://racer5-cobot_description/meshes/racer5-cobot/Link4.STL" />
@@ -131,5 +132,5 @@
     </link>
     <joint name="${prefix}joint_4" type="revolute">
-      <origin xyz="-0.049998 0 0.121" rpy="0 0 0" />
+      <origin xyz="0.05 0 0.0" rpy="0 0 0" />
       <parent link="link_3" />
       <child link="link_4" />
@@ -158,5 +159,5 @@
     </link>
     <joint name="${prefix}joint_5" type="revolute">
-      <origin xyz="0 0 0.26494" rpy="0 0 0" />
+      <origin xyz="0 0 0.38594" rpy="0 0 0" />
       <parent link="link_4" />
       <child link="link_5" />
@@ -186,10 +187,10 @@
       </collision>
     </link>
-    <joint name="${prefix}joint_6" type="revolute"> <!--"continuous"-->
-      <origin xyz="0 0 0.0665" rpy="0 0 0" />
+    <joint name="${prefix}joint_6" type="revolute">
+      <origin xyz="0 0 0.08" rpy="0 0 0" />
       <parent link="link_5" />
       <child link="link_6" />
       <axis xyz="0 0 -1" />
-      <limit lower="-47.10" upper="47.10" effort="100000.00" velocity="20.00" />
+      <limit lower="-100" upper="100" effort="100000.00" velocity="20.00" />
     </joint>
     <link name="${prefix}ee_link">
@@ -201,5 +202,5 @@
     </link>
     <joint name="${prefix}joint_ee_link" type="fixed">
-      <origin xyz="0.0 0.0 0.0" rpy="0 0 0.0"/>
+      <origin xyz="0.0 0.0 0.0" rpy="0 0 3.14"/>
       <parent link="link_6"/>
       <child link="ee_link"/>
