Commit message: racer5-cobot description converted from urdf.xacro to urdf

File: comau_ros2_client/comau_description/racer5-cobot_description/urdf/racer5-cobot/racer5-cobot_robot.urdf (robot description, URDF)
Before this commit: robot racer5-cobot, 9 links, 8 joints
Joints:
- joint joint_1: axis 0 0 1 -> 0 0 -1; origin xyz=0 0 0.1895 rpy=0 0 0 -> xyz=0 0 0.242 rpy=0 0 0
- joint joint_2: axis 0 -1 0 -> 0 1 0; limit lower=-1.99 upper=1.116 effort=100000.00 velocity=20.00 -> lower=-1.116 upper=1.99 effort=100000.00 velocity=20.00; origin xyz=0.05 0 0.1755 rpy=0 0 0 -> xyz=0.05 0 0.123 rpy=0 0 0
- joint joint_3: axis 0 -1 0 -> 0 1 0; origin xyz=0 0 0.37 rpy=0 0 0 -> xyz=0 0 0.37 rpy=0 0 3.14
- joint joint_4: origin xyz=-0.049998 0 0.121 rpy=0 0 0 -> xyz=0.05 0 0.0 rpy=0 0 0
- joint joint_5: origin xyz=0 0 0.26494 rpy=0 0 0 -> xyz=0 0 0.38594 rpy=0 0 0
- joint joint_6: limit lower=-47.10 upper=47.10 effort=100000.00 velocity=20.00 -> lower=-100 upper=100 effort=100000.00 velocity=20.00; origin xyz=0 0 0.0665 rpy=0 0 0 -> xyz=0 0 0.08 rpy=0 0 0
- joint joint_ee_link: origin xyz=0.0 0.0 0.0 rpy=0 0 0.0 -> xyz=0.0 0.0 0.0 rpy=0 0 3.14
