Commit message: Update URDF Moveing

File: comau_ros2_client/comau_description/racer5-cobot_description/robots/racer5-cobot_robot.urdf.xacro (robot description, xacro)
@@ -1,25 +1,6 @@
 <?xml version="1.0"?>
-<robot xmlns:xacro="http://wiki.ros.org/xacro" name="racer5-cobot">
-  <!--
-    Author: LMS
-   -->
-  <xacro:arg name="transmission_hw_interface" default="hardware_interface/PositionJointInterface"/>
-  <xacro:arg name="pos_x" default="0"/>
-  <xacro:arg name="pos_y" default="0"/>
-  <xacro:arg name="pos_z" default="0"/>
-  <xacro:arg name="roll" default="0"/>
-  <xacro:arg name="pitch" default="0"/>
-  <xacro:arg name="yaw" default="0"/>
-  <!-- common stuff -->
-  <xacro:include filename="$(find racer5-cobot_description)/urdf/common.gazebo.xacro" />
+<robot xmlns:xacro="http://www.ros.org/wiki/xacro" name="racer5-cobot">
   <!--load racer5-cobot -->
   <xacro:include filename="$(find racer5-cobot_description)/urdf/racer5-cobot/racer5-cobot.urdf.xacro" />
-  <!-- arm -->
-  <xacro:racer5-cobot_robot prefix="" transmission_hw_interface="$(arg transmission_hw_interface)"/>
-  <link name="world" />
-  <joint name="world_joint" type="fixed">
-    <parent link="world" />
-    <child link = "base_link" />
-    <origin xyz="$(arg pos_x) $(arg pos_y) $(arg pos_z)" rpy="$(arg roll) $(arg pitch) $(arg yaw)" />
-  </joint>
+  <xacro:racer5_cobot_description/>
 </robot>

File: comau_ros2_client/comau_description/racer5-cobot_description/urdf/comau_common.macro.xacro (robot description, xacro)
@@ -1,4 +1,4 @@
 <?xml version="1.0"?>
-<robot xmlns:xacro="http://wiki.ros.org/xacro">
+<robot xmlns:xacro="http://www.ros.org/wiki/xacro">
   <!-- colors -->
   <xacro:macro name="c_d_grey">

File: comau_ros2_client/comau_description/racer5-cobot_description/urdf/racer5-cobot/racer5-cobot.urdf.xacro (robot description, xacro)
@@ -1,14 +1,12 @@
 <?xml version="1.0"?>
-<robot xmlns:xacro="http://wiki.ros.org/xacro">
-  <!--
-    Author: LMS
-   -->
-  <xacro:include filename="$(find racer5-cobot_description)/urdf/comau_common.macro.xacro" />
-  <xacro:include filename="$(find racer5-cobot_description)/urdf/racer5-cobot/racer5-cobot.transmission.xacro" />
+<robot xmlns:xacro="http://www.ros.org/wiki/xacro">
+  <xacro:macro name="racer5_cobot_description">
+   <xacro:include filename="$(find racer5-cobot_description)/urdf/comau_common.macro.xacro" />
+  <!--xacro:include filename="$(find racer5-cobot_description)/urdf/racer5-cobot/racer5-cobot.transmission.xacro" />
   <xacro:include filename="$(find racer5-cobot_description)/urdf/racer5-cobot/racer5-cobot.gazebo.xacro" />
   <xacro:macro name="racer5-cobot_robot" params="prefix transmission_hw_interface:=hardware_interface/PositionJointInterface">
     <xacro:racer5-cobot_transmission prefix="${prefix}" hw_interface="${transmission_hw_interface}" />
-    <xacro:racer5-cobot_gazebo prefix="${prefix}" />
-    <link name="${prefix}base_link">
+    <xacro:racer5-cobot_gazebo prefix="${prefix}" /-->
+    <link name="base_link">
       <inertial>
         <origin xyz="-0.017279 0.00078009 0.14492" rpy="0 0 0" />
@@ -21,5 +19,5 @@
           <mesh filename="package://racer5-cobot_description/meshes/racer5-cobot/base_link.STL" />
         </geometry>
-        <xacro:c_d_grey/>
+        <xacro:c_white/>
       </visual>
       <collision>
@@ -30,5 +28,5 @@
       </collision>
     </link>
-    <link name="${prefix}link_1">
+    <link name="link_1">
       <inertial>
         <origin xyz="0.0375246972830294 -0.0047330722058841 0.119959023209445" rpy="0 0 0" />
@@ -41,5 +39,5 @@
           <mesh filename="package://racer5-cobot_description/meshes/racer5-cobot/Link1.STL" />
         </geometry>
-        <xacro:c_white/>
+        <xacro:c_blue/>
       </visual>
       <collision>
@@ -50,5 +48,5 @@
       </collision>
     </link>
-    <joint name="${prefix}joint_1" type="revolute">
+    <joint name="joint_1" type="revolute">
       <origin xyz="0 0 0.242" rpy="0 0 0" />
       <parent link="base_link" />
@@ -68,5 +66,5 @@
           <mesh filename="package://racer5-cobot_description/meshes/racer5-cobot/Link2.STL" />
         </geometry>
-        <xacro:c_blue/>
+        <xacro:c_white/>
       </visual>
       <collision>
@@ -77,5 +75,5 @@
       </collision>
     </link>
-    <joint name="${prefix}joint_2" type="revolute">
+    <joint name="joint_2" type="revolute">
       <origin xyz="0.05 0 0.123" rpy="0 0 0" />
       <parent link="link_1" />
@@ -84,5 +82,5 @@
       <limit lower="-1.116" upper="1.99" effort="100000.00" velocity="20.00" />
     </joint>
-    <link name="${prefix}link_3">
+    <link name="link_3">
       <inertial>
         <origin xyz="-0.0174695057689258 -0.00108883931260707 -0.00846478214002855" rpy="0 0 0" />
@@ -95,5 +93,5 @@
           <mesh filename="package://racer5-cobot_description/meshes/racer5-cobot/Link3.STL" />
         </geometry>
-         <xacro:c_white/>
+         <xacro:c_blue/>
       </visual>
       <collision>
@@ -104,5 +102,5 @@
       </collision>
     </link>
-    <joint name="${prefix}joint_3" type="revolute">
+    <joint name="joint_3" type="revolute">
       <origin xyz="0 0 0.37" rpy="0 0 3.14" />
       <parent link="link_2" />
@@ -111,5 +109,5 @@
       <limit lower="-2.62" upper="1.483" effort="100000.00" velocity="20.00" />
     </joint>
-    <link name="${prefix}link_4">
+    <link name="link_4">
       <inertial>
         <origin xyz="-0.00227788070042482 -0.00123420975347735 0.0624227170360064" rpy="0 0 0" />
@@ -118,9 +116,9 @@
       </inertial>
       <visual>
-        <origin xyz="0 0 0" rpy="0 0 3.14" />
+        <origin xyz="0 0 0.125" rpy="0 0 3.14" />
         <geometry>
           <mesh filename="package://racer5-cobot_description/meshes/racer5-cobot/Link4.STL" />
         </geometry>
-        <xacro:c_blue/>
+        <xacro:c_white/>
       </visual>
       <collision>
@@ -131,5 +129,5 @@
       </collision>
     </link>
-    <joint name="${prefix}joint_4" type="revolute">
+    <joint name="joint_4" type="revolute">
       <origin xyz="0.05 0 0.0" rpy="0 0 0" />
       <parent link="link_3" />
@@ -138,5 +136,5 @@
       <limit lower="-3.49" upper="3.49" effort="100000.00" velocity="20.00" />
     </joint>
-    <link name="${prefix}link_5">
+    <link name="link_5">
       <inertial>
         <origin xyz="8.42234791683474E-06 0.000438242230281476 0.0364200996149726" rpy="0 0 0" />
@@ -149,5 +147,5 @@
           <mesh filename="package://racer5-cobot_description/meshes/racer5-cobot/Link5.STL" />
         </geometry>
-        <xacro:c_white/>
+        <xacro:c_blue/>
       </visual>
       <collision>
@@ -158,5 +156,5 @@
       </collision>
     </link>
-    <joint name="${prefix}joint_5" type="revolute">
+    <joint name="joint_5" type="revolute">
       <origin xyz="0 0 0.38594" rpy="0 0 0" />
       <parent link="link_4" />
@@ -165,5 +163,5 @@
       <limit lower="-1.83" upper="1.83" effort="100000.00" velocity="20.00" />
     </joint>
-    <link name="${prefix}link_6">
+    <link name="link_6">
       <inertial>
         <origin xyz="5.64165774402925E-05 -4.33361315668251E-07 0.00365583421206228" rpy="0 0 0" />
@@ -172,5 +170,5 @@
       </inertial>
       <visual>
-        <xacro:c_d_grey/>
+        <xacro:c_white/>
         <geometry>
           <mesh filename="package://racer5-cobot_description/meshes/racer5-cobot/Link6.STL" />
@@ -187,5 +185,5 @@
       </collision>
     </link>
-    <joint name="${prefix}joint_6" type="revolute">
+    <joint name="joint_6" type="revolute">
       <origin xyz="0 0 0.08" rpy="0 0 0" />
       <parent link="link_5" />
@@ -194,5 +192,5 @@
       <limit lower="-100" upper="100" effort="100000.00" velocity="20.00" />
     </joint>
-    <link name="${prefix}ee_link">
+    <link name="ee_link">
       <visual>
         <geometry>
@@ -201,5 +199,5 @@
       </visual>
     </link>
-    <joint name="${prefix}joint_ee_link" type="fixed">
+    <joint name="joint_ee_link" type="fixed">
       <origin xyz="0.0 0.0 0.0" rpy="0 0 3.14"/>
       <parent link="link_6"/>
