Commit message: changed edo base

File: comau_ros2_client/comau_description/edo_description/urdf/edo/edo.urdf.xacro (robot description, xacro)
@@ -26,9 +26,9 @@
             <visual>
        <origin
-		  xyz="0 0 0.135"
+		  xyz="0 0 0.0"
 		  rpy="0 0 0"/>
        <geometry>
  	<mesh
-	  filename="package://edo_description/meshes/visual/link_0.dae"/>
+	  filename="package://edo_description/meshes/visual/base_link.STL"/>
        </geometry>
        <material
@@ -38,5 +38,5 @@
                 <origin xyz="0 0 0.135" rpy="0 0 0"/>
                 <geometry>
-                    <mesh filename="package://edo_description/meshes/collision/link_0.dae"/>
+                    <mesh filename="package://edo_description/meshes/collision/base_link.STL"/>
                 </geometry>
             </collision>

Commit message: Added the 7th joint to eDo

File: comau_ros2_client/comau_description/edo_description/urdf/edo/edo.urdf.xacro (robot description, xacro)
@@ -392,4 +392,15 @@
       <child link="ee_link"/>
   </joint>
+  <link name="tool" />
+  <joint name="tool_joint" type="revolute">
+     <origin
+      xyz="0.0 0 0.0"
+      rpy="1.57 0 1.57" />
+    <parent link="ee_link" />
+    <child link = "tool" />
+    <axis
+       xyz="0 0 1"/>
+    <limit lower="-3.14" upper="3.14" effort="100000.00" velocity="20.00" />
+  </joint>
   </xacro:macro>
 </robot>
